Commit message: update custom_bot.xacro: wheels and caster

File: custom_bot/urdf/custom_bot.xacro (robot description, xacro)
@@ -11,5 +11,5 @@
     <pose>0 0 0.1 0 0 0</pose>
     <inertial>
-      <mass value="15.0"/>
+      <mass value="10.0"/>
       <origin xyz="0.0 0 0" rpy=" 0 0 0"/>
       <inertia
@@ -23,5 +23,5 @@
       <geometry>
         <!-- box size=".4 .2 .1"/ -->
-        <cylinder radius="0.5" length="0.1"/>
+        <cylinder radius="0.3" length="0.1"/>
       </geometry>
     </collision>
@@ -30,9 +30,9 @@
       <geometry>
         <!-- box size=".4 .2 .1"/ -->
-        <cylinder radius="0.5" length="0.1"/>
+        <cylinder radius="0.3" length="0.1"/>
       </geometry>
     </visual>
     <collision name='back_caster_collision'>
-      <origin xyz="-0.15 0 -0.05" rpy=" 0 0 0"/>
+      <origin xyz="-0.25 0 -0.05" rpy=" 0 0 0"/>
       <geometry>
         <sphere radius="0.05"/>
@@ -50,27 +50,5 @@
     </collision>
     <visual name='back_caster_visual'>
-      <origin xyz="-0.15 0 -0.05" rpy=" 0 0 0"/>
-      <geometry>
-        <sphere radius="0.05"/>
-      </geometry>
-    </visual>
-    <collision name='front_caster_collision'>
-      <origin xyz="0.15 0 -0.05" rpy=" 0 0 0"/>
-      <geometry>
-        <sphere radius="0.05"/>
-      </geometry>
-      <surface>
-        <friction>
-          <ode>
-            <mu>0</mu>
-            <mu2>0</mu2>
-            <slip1>1.0</slip1>
-            <slip2>1.0</slip2>
-          </ode>
-        </friction>
-      </surface>
-    </collision>
-    <visual name='front_caster_visual'>
-      <origin xyz="0.15 0 -0.05" rpy=" 0 0 0"/>
+      <origin xyz="-0.25 0 -0.05" rpy=" 0 0 0"/>
       <geometry>
         <sphere radius="0.05"/>
@@ -79,5 +57,5 @@
   </link>
   <joint type="continuous" name="left_wheel_hinge">
-    <origin xyz="0 0.15 0" rpy="0 0 0"/>
+    <origin xyz="0.15 0.15 -0.05" rpy="0 0 0"/>
     <child link="left_wheel"/>
     <parent link="chassis"/>
@@ -99,5 +77,5 @@
       <origin xyz="0 0 0" rpy="0 1.5707 1.5707"/>
       <geometry>
-        <cylinder radius="0.1" length="0.05"/>
+        <cylinder radius="0.05" length="0.05"/>
       </geometry>
     </collision>
@@ -105,10 +83,10 @@
       <origin xyz="0 0 0" rpy="0 1.5707 1.5707"/>
       <geometry>
-        <cylinder radius="0.1" length="0.05"/>
+        <cylinder radius="0.05" length="0.05"/>
       </geometry>
     </visual>
   </link>
   <joint type="continuous" name="right_wheel_hinge">
-    <origin xyz="0 -0.15 0" rpy="0 0 0"/>
+    <origin xyz="0.15 -0.15 -0.05" rpy="0 0 0"/>
     <child link="right_wheel"/>
     <parent link="chassis"/>
@@ -130,5 +108,5 @@
       <origin xyz="0 0 0" rpy="0 1.5707 1.5707"/>
       <geometry>
-        <cylinder radius="0.1" length="0.05"/>
+        <cylinder radius="0.05" length="0.05"/>
       </geometry>
     </collision>
@@ -136,5 +114,5 @@
       <origin xyz="0 0 0" rpy="0 1.5707 1.5707"/>
       <geometry>
-        <cylinder radius="0.1" length="0.05"/>
+        <cylinder radius="0.05" length="0.05"/>
       </geometry>
     </visual>

Commit message: update custom_bot.xacro: camera and rangefinder positions

File: custom_bot/urdf/custom_bot.xacro (robot description, xacro)
@@ -66,5 +66,5 @@
   <link name='left_wheel'>
     <inertial>
-      <mass value="5.0"/>
+      <mass value="1.0"/>
       <origin xyz="0 0 0" rpy="0 1.5707 1.5707"/>
       <inertia
@@ -97,5 +97,5 @@
   <link name='right_wheel'>
     <inertial>
-      <mass value="5.0"/>
+      <mass value="1.0"/>
       <origin xyz="0 0 0" rpy="0 1.5707 1.5707"/>
       <inertia
@@ -119,5 +119,5 @@
   </link>
   <joint type="fixed" name="camera_joint">
-    <origin xyz="0.2 0 0" rpy="0 0 0"/>
+    <origin xyz="0.275 0 0" rpy="0 0 0"/>
     <child link="camera"/>
     <parent link="chassis"/>
@@ -150,5 +150,5 @@
   </link>
   <joint type="fixed" name="hokuyo_joint">
-    <origin xyz="0.15 0 0.1" rpy="0 0 0"/>
+    <origin xyz="0 0 0.1" rpy="0 0 0"/>
     <child link="hokuyo"/>
     <parent link="chassis"/>

Commit message: add color to custom_bot

File: custom_bot/urdf/custom_bot.xacro (robot description, xacro)
@@ -30,4 +30,7 @@
         <cylinder radius="0.3" length="0.1"/>
       </geometry>
+      <material name='chassis_color'>
+        <color rgba="0.6 0.8 0.88 1"/>
+      </material>
     </visual>
     <collision name='back_caster_collision'>
@@ -83,4 +86,7 @@
         <cylinder radius="0.05" length="0.05"/>
       </geometry>
+      <material name='left_wheel_color'>
+        <color rgba="0.75 0 0.75 1"/>
+      </material>
     </visual>
   </link>
@@ -114,4 +120,7 @@
         <cylinder radius="0.05" length="0.05"/>
       </geometry>
+      <material name='right_wheel_color'>
+        <color rgba="0.75 0 0.75 1"/>
+      </material>
     </visual>
   </link>
@@ -145,4 +154,7 @@
         <box size="0.05 0.05 0.05"/>
       </geometry>
+      <material name='camera_color'>
+        <color rgba="0 1 0.75294 1"/>
+      </material>
     </visual>
   </link>

Commit message: split amcl.yaml and update parameters for custom_bot

File: custom_bot/urdf/custom_bot.xacro (robot description, xacro)
@@ -22,5 +22,5 @@
       <origin xyz="0 0 0" rpy=" 0 0 0"/>
       <geometry>
-        <cylinder radius="0.3" length="0.1"/>
+        <cylinder radius="0.25" length="0.1"/>
       </geometry>
     </collision>
@@ -28,5 +28,5 @@
       <origin xyz="0 0 0" rpy=" 0 0 0"/>
       <geometry>
-        <cylinder radius="0.3" length="0.1"/>
+        <cylinder radius="0.25" length="0.1"/>
       </geometry>
       <material name='chassis_color'>
@@ -35,5 +35,5 @@
     </visual>
     <collision name='back_caster_collision'>
-      <origin xyz="-0.25 0 -0.05" rpy=" 0 0 0"/>
+      <origin xyz="-0.2 0 -0.05" rpy=" 0 0 0"/>
       <geometry>
         <sphere radius="0.05"/>
@@ -51,5 +51,5 @@
     </collision>
     <visual name='back_caster_visual'>
-      <origin xyz="-0.25 0 -0.05" rpy=" 0 0 0"/>
+      <origin xyz="-0.2 0 -0.05" rpy=" 0 0 0"/>
       <geometry>
         <sphere radius="0.05"/>
@@ -58,5 +58,5 @@
   </link>
   <joint type="continuous" name="left_wheel_hinge">
-    <origin xyz="0.15 0.15 -0.05" rpy="0 0 0"/>
+    <origin xyz="0.15 0.2 -0.05" rpy="0 0 0"/>
     <child link="left_wheel"/>
     <parent link="chassis"/>
@@ -92,5 +92,5 @@
   </link>
   <joint type="continuous" name="right_wheel_hinge">
-    <origin xyz="0.15 -0.15 -0.05" rpy="0 0 0"/>
+    <origin xyz="0.15 -0.2 -0.05" rpy="0 0 0"/>
     <child link="right_wheel"/>
     <parent link="chassis"/>
@@ -126,5 +126,5 @@
   </link>
   <joint type="fixed" name="camera_joint">
-    <origin xyz="0.275 0 0" rpy="0 0 0"/>
+    <origin xyz="0.225 0 0" rpy="0 0 0"/>
     <child link="camera"/>
     <parent link="chassis"/>
@@ -160,5 +160,5 @@
   </link>
   <joint type="fixed" name="hokuyo_joint">
-    <origin xyz="0 0 0.1" rpy="0 0 0"/>
+    <origin xyz="0.15 0 0.1" rpy="0 0 0"/>
     <child link="hokuyo"/>
     <parent link="chassis"/>

Commit message: rotate camera in urdf

File: custom_bot/urdf/custom_bot.xacro (robot description, xacro)
@@ -2,4 +2,5 @@
 <robot name="custom_bot" xmlns:xacro="http://www.ros.org/wiki/xacro">
   <xacro:include filename="$(find custom_bot)/urdf/custom_bot.gazebo" />
+  <xacro:property name="M_PI" value="3.1415926535897931" />
   <link name="robot_footprint"></link>
   <joint name="robot_footprint_joint" type="fixed">
@@ -159,4 +160,11 @@
     </visual>
   </link>
+  <joint name="camera_optical_joint" type="fixed">
+    <origin xyz="0 0 0" rpy="${-M_PI/2} 0 ${-M_PI/2}" />
+    <parent link="camera" />
+    <child link="camera_optical" />
+  </joint>
+  <link name="camera_optical">
+  </link>
   <joint type="fixed" name="hokuyo_joint">
     <origin xyz="0.15 0 0.1" rpy="0 0 0"/>
